Commit message: Fixed simulation with ros2 launch. Pedestrians moves

File: rb_theron_description_fortress/robots/rb_theron.urdf.xacro (robot description, xacro)
@@ -11,4 +11,5 @@
 	<xacro:include filename="$(find rb_theron_description_fortress)/urdf/wheels/rubber_wheel_150.urdf.xacro" />
 	<!-- Import all available sensors -->
+	<xacro:include filename="$(find rb_theron_description_fortress)/urdf/sensors/imu.urdf.xacro" />
 	<xacro:include filename="$(find rb_theron_description_fortress)/urdf/common.gazebo.xacro" />
 	<!-- Import Gazebo Stuff -->
@@ -40,5 +41,5 @@
 	<!-- Gazebo ros control pluggins -->
 	<!--xacro:ros_control namespace="$(arg namespace)"/-->
-	<xacro:ros_control/>
+	<!-- <xacro:ros_control/> -->
 	<xacro:if value="$(arg ros_planar_move_plugin)">
     	<xacro:omni_steering prefix="$(arg prefix)" publish_tf="true"/>
@@ -46,4 +47,7 @@
 	<xacro:gazebo_colors prefix="$(arg prefix)"/>
 <!-- SENSORS -->
+	<xacro:imu_sensor prefix="$(arg prefix)" parent="$(arg prefix)base_link"/>
+	<xacro:include filename="$(find rb_theron_description_fortress)/urdf/sensors/laser_sensor.urdf.xacro" />
+	<xacro:laser_sensor prefix="$(arg prefix)" parent="$(arg prefix)base_link"/>
 <!--
   TODO: Moved 0.01 in x, otherwise the camera is still inside the robot
@@ -76,3 +80,31 @@
 	</xacro:sensor_sick_tim571>
 	-->
+    <gazebo>
+        <plugin filename="libgz_ros2_control-system.so" name="gz_ros2_control::GazeboSimSystem">
+            <robot_param>robot_description</robot_param>
+            <robot_param_node>robot_state_publisher</robot_param_node>
+            <parameters>$(find rb_theron_description_fortress)/config/controllers.yaml</parameters>
+        </plugin>
+    </gazebo>
+    <ros2_control name="GazeboSystem" type="system">
+        <hardware>
+            <plugin>gz_ros2_control/GazeboSimSystem</plugin>
+        </hardware>
+        <joint name="robot_left_wheel_joint">
+            <command_interface name="velocity">
+                <param name="min">-10</param>
+                <param name="max">10</param>
+            </command_interface>
+            <state_interface name="position" />
+            <state_interface name="velocity" />
+        </joint>
+        <joint name="robot_right_wheel_joint">
+            <command_interface name="velocity">
+                <param name="min">-10</param>
+                <param name="max">10</param>
+            </command_interface>
+            <state_interface name="position" />
+            <state_interface name="velocity" />
+        </joint>
+    </ros2_control>
 </robot>

File: rb_theron_description_fortress/urdf/bases/base.gazebo.xacro (robot description, xacro)
@@ -3,4 +3,5 @@
   <!-- ros control plugin -->
   <xacro:macro name="ros_control">
+    <!--
     <gazebo>
       <plugin name="ros_control" filename="libgazebo_ros_control.so">
@@ -11,4 +12,5 @@
       </plugin>
     </gazebo>
+    -->
 	</xacro:macro>
 	<!-- skid steering plugin -->
